Commit message: first commit

File: urdf/control.xacro (robot description, xacro)
@@ -1,32 +1,72 @@
 <?xml version="1.0"?>
 <robot name="gypsy" xmlns:xacro="http://www.ros.org/wiki/xacro">
-    <ros2_control name="MecanumWheelSystem" type="system">
-        <hardware>
-            <plugin>gazebo_ros2_control/MecanumWheelSystem</plugin>
-        </hardware>
-        <joint name="upper_left_wheel_joint">
-            <command_interface name="velocity"/>
-            <state_interface name = "position"/>
-            <state_interface name = "velocity"/>
-            <param name="motor_id">1</param>
-        </joint>
-        <joint name="bottom_left_wheel_joint">
-            <command_interface name="velocity"/>
-            <state_interface name = "position"/>
-            <state_interface name = "velocity"/>
-            <param name="motor_id">2</param>
-        </joint>
-        <joint name="upper_right_wheel_joint">
-            <command_interface name="velocity"/>
-            <state_interface name = "position"/>
-            <state_interface name = "velocity"/>
-            <param name="motor_id">3</param>
-        </joint>
-        <joint name="bottom_right_wheel_joint">
-            <command_interface name="velocity"/>
-            <state_interface name = "position"/>
-            <state_interface name = "velocity"/>
-            <param name="motor_id">4</param>
-        </joint>
-    </ros2_control>
+  <ros2_control name="MecanumWheelSystem" type="system">
+    <hardware>
+      <plugin>gazebo_ros2_control/MecanumWheelSystem</plugin>
+    </hardware>
+    <joint name="upper_left_wheel_joint">
+      <command_interface name="velocity"/>
+      <state_interface name = "position"/>
+      <state_interface name = "velocity"/>
+      <param name="motor_id">1</param>
+    </joint>
+    <joint name="bottom_left_wheel_joint">
+      <command_interface name="velocity"/>
+      <state_interface name = "position"/>
+      <state_interface name = "velocity"/>
+      <param name="motor_id">2</param>
+    </joint>
+    <joint name="upper_right_wheel_joint">
+      <command_interface name="velocity"/>
+      <state_interface name = "position"/>
+      <state_interface name = "velocity"/>
+      <param name="motor_id">3</param>
+    </joint>
+    <joint name="bottom_right_wheel_joint">
+      <command_interface name="velocity"/>
+      <state_interface name = "position"/>
+      <state_interface name = "velocity"/>
+      <param name="motor_id">4</param>
+    </joint>
+  </ros2_control>
+  <transmission name="front_left_wheel_trans" type="SimpleTransmission">
+    <type>transmission_interface/SimpleTransmission</type>
+    <actuator name="front_left_wheel_motor">
+      <hardwareInterface>hardware_interface/VelocityJointInterface</hardwareInterface>
+      <mechanicalReduction>1</mechanicalReduction>
+    </actuator>
+    <joint name="upper_left_wheel_joint">
+      <hardwareInterface>hardware_interface/VelocityJointInterface</hardwareInterface>
+    </joint>
+  </transmission>
+  <transmission name="front_right_wheel_trans" type="SimpleTransmission">
+    <type>transmission_interface/SimpleTransmission</type>
+    <actuator name="front_right_wheel_motor">
+      <hardwareInterface>hardware_interface/VelocityJointInterface</hardwareInterface>
+      <mechanicalReduction>1</mechanicalReduction>
+    </actuator>
+    <joint name="bottom_left_wheel_joint">
+      <hardwareInterface>hardware_interface/VelocityJointInterface</hardwareInterface>
+    </joint>
+  </transmission>
+  <transmission name="rear_left_wheel_trans" type="SimpleTransmission">
+    <type>transmission_interface/SimpleTransmission</type>
+    <actuator name="rear_left_wheel_motor">
+      <hardwareInterface>hardware_interface/VelocityJointInterface</hardwareInterface>
+      <mechanicalReduction>1</mechanicalReduction>
+    </actuator>
+    <joint name="upper_right_wheel_joint">
+      <hardwareInterface>hardware_interface/VelocityJointInterface</hardwareInterface>
+    </joint>
+  </transmission>
+  <transmission name="rear_right_wheel_trans" type="SimpleTransmission">
+    <type>transmission_interface/SimpleTransmission</type>
+    <actuator name="rear_right_wheel_motor">
+      <hardwareInterface>hardware_interface/VelocityJointInterface</hardwareInterface>
+      <mechanicalReduction>1</mechanicalReduction>
+    </actuator>
+    <joint name="bottom_right_wheel_joint">
+      <hardwareInterface>hardware_interface/VelocityJointInterface</hardwareInterface>
+    </joint>
+  </transmission>
 </robot>

File: urdf/gypsy.urdf.xacro (robot description, xacro)
@@ -7,4 +7,6 @@
     <xacro:include filename ="$(find gypsy_robot)/urdf/gazebo_description/material.gazebo"/>
     <xacro:include filename ="$(find gypsy_robot)/urdf/gazebo_description/plugin.gazebo"/>
+    <xacro:include filename ="$(find gypsy_robot)/urdf/gazebo_description/physics.gazebo"/>
+    <!--########################################################################################-->
     <link name = "base_footprint"></link>
     <joint name="base_link_joint" type="fixed">

File: urdf/gypsy_mobile.urdf.xacro (robot description, xacro)
@@ -28,8 +28,9 @@
             <origin xyz="0 0 0" rpy="0 0 0"/>
             <mass value = "30.00"/>
+            <!--calcuated on the basis of dimension-->
             <inertia
-                ixx = "1.66" ixy="0.00" ixz="-0.001"
-                iyy = "0.00" iyz="0.0004555"
-                izz = "3.383"/>
+                ixx = "3.355625" ixy="0.00" ixz="0.00"
+                iyy = "1.40" iyz="0.0004555"
+                izz = "2.825"/>
         </inertial>
     </link>
@@ -108,9 +109,9 @@
             <inertial>
                 <origin xyz = "0 0 0" rpy="0 0 0"/>
-                <mass value = "2.883"/>
+                <mass value = "0.200"/>
                 <inertia
-                    ixx = "0.047" ixy="0.00" ixz="0.00"
-                    iyy = "0.074" iyz="0.0"
-                    izz = "0.051"/>
+                    ixx = "0.004" ixy="0.00" ixz="0.00"
+                    iyy = "0.004" iyz="0.0"
+                    izz = "0.004"/>
             </inertial>
         </link>
