Commit message: added supermarket world and made slight changes in urdf and sdf files

File: urdf/gypsy.urdf (robot description, URDF)
Before this commit: robot gypsy, 23 links, 22 joints
Links:
- link bin_green: mass 2.883 -> 0.200
- link bin_red: mass 2.883 -> 0.200

File: urdf/gypsy.urdf.xacro (robot description, xacro)
@@ -1,4 +1,5 @@
 <?xml version="1.0"?>
 <robot name="gypsy" xmlns:xacro="http://ros.org/wiki/xacro">
+    <xacro:property name ="PI" value="3.1415926535897931"/>
     <xacro:include filename="$(find gypsy_robot)/urdf/panda.xacro"/>
     <xacro:include filename="$(find gypsy_robot)/urdf/gypsy_mobile.urdf.xacro"/>

File: urdf/gypsy_mobile.urdf.xacro (robot description, xacro)
@@ -30,6 +30,6 @@
             <!--calcuated on the basis of dimension-->
             <inertia
-                ixx = "3.355625" ixy="0.00" ixz="0.00"
-                iyy = "1.40" iyz="0.0004555"
+                ixx = "1.7755" ixy="0.00" ixz="0.00"
+                iyy = "1.40" iyz="0.00"
                 izz = "2.825"/>
         </inertial>

Commit message: updates plugins values

File: urdf/gypsy.urdf (robot description, URDF)
Before this commit: robot gypsy, 23 links, 22 joints
Links:
- added link laser_link; visual box size=0.001 0.001 0.001
Joints:
- added joint laser_link_joint: type fixed, parent camera_one, child laser_link, origin xyz=0 0 0 rpy=1.57 -1.57 0

File: urdf/gypsy_mobile.urdf.xacro (robot description, xacro)
@@ -147,4 +147,13 @@
     <xacro:camera prefix="one"/>
     <xacro:camera prefix = "two"/>
+    <!--##################### LASER Link ####################-->
+    <link name="laser_link">
+        <visual>
+            <origin xyz="0 0 0" rpy="0 0 0"/>
+            <geometry>
+                <box size="0.1 0.02 0.01"/>
+            </geometry>
+        </visual>
+    </link>
     <!--##################### IMU Link ####################-->
     <link name="imu_link">
@@ -204,3 +213,8 @@
         <origin xyz="0 0 0" rpy="0 0 0"/>
     </joint>
+    <joint name="laser_link_joint" type="fixed">
+        <parent link="camera_one" />
+        <child link="laser_link" />
+        <origin xyz="0 0 0" rpy="0 0 0"/>
+    </joint>
 </robot>
