Commit message: minor fixes

File: urdf/gypsy.urdf.xacro (robot description, xacro)
@@ -4,5 +4,4 @@
     <xacro:include filename="$(find gypsy_robot)/urdf/panda.xacro"/>
     <xacro:include filename="$(find gypsy_robot)/urdf/gypsy_mobile.urdf.xacro"/>
-    <xacro:include filename="$(find gypsy_robot)/urdf/control.xacro"/>
     <xacro:include filename ="$(find gypsy_robot)/urdf/gazebo_description/panda.gazebo"/>
     <xacro:include filename ="$(find gypsy_robot)/urdf/gazebo_description/material.gazebo"/>

File: urdf/gypsy_mobile.urdf.xacro (robot description, xacro)
@@ -152,5 +152,5 @@
             <origin xyz="0 0 0" rpy="0 0 0"/>
             <geometry>
-                <box size="0.1 0.02 0.01"/>
+                <box size="0.001 0.001 0.001"/>
             </geometry>
         </visual>
@@ -216,5 +216,5 @@
         <parent link="camera_one" />
         <child link="laser_link" />
-        <origin xyz="0 0 0" rpy="0 0 0"/>
+        <origin xyz="1.57 -1.57 0" rpy="0 0 0"/>
     </joint>
 </robot>
